File: relay.kicad_sch (KiCad schematic)
At the start: 5 parts, among them J44 Conn_01x08_Pin, U16 ULN2803A, U26 SN74LVC245APW

Commit message: added lcsc field so that bom can match during jlcpcb fab
Parts:
- C56: LCSC (none) -> C15849
- C80: LCSC (none) -> C14663
- J44: LCSC (none) -> C2894931
- U16: LCSC (none) -> C845537
- U26: LCSC (none) -> C5980
Changed lines of the file:
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@@
+			)
+		)
+		(property "LCSC" "C15849"
+			(at 156.21 53.34 0)
+			(effects
+				(font
+					(size 1.27 1.27)
+				)
+				(hide yes)
 			)
 		)
@@
 			)
 		)
+		(property "LCSC" "C5980"
+			(at 67.31 57.15 0)
+			(effects
+				(font
+					(size 1.27 1.27)
+				)
+				(hide yes)
+			)
+		)
 		(pin "16"
 		)
@@
 		)
 		(property "Tape" "8x4"
+			(at 25.4 24.13 0)
+			(effects
+				(font
+					(size 1.27 1.27)
+				)
+				(hide yes)
+			)
+		)
+		(property "LCSC" "C14663"
 			(at 25.4 24.13 0)
 			(effects
@@
 			)
 		)
+		(property "LCSC" "C2894931"
+			(at 91.44 85.09 0)
+			(effects
+				(font
+					(size 1.27 1.27)
+				)
+				(hide yes)
+			)
+		)
 		(pin "5"
 		)
@@
 			(at 130.81 57.15 0)
 			(effects
+				(font
+					(size 1.27 1.27)
+				)
+				(hide yes)
+			)
+		)
+		(property "LCSC" "C845537"
+			(at 130.81 57.15 0)
+			(effects
