File: rs485.kicad_sch (KiCad schematic)
At the start: 3 parts, among them U2 MAX3078E

Commit message: added lcsc field so that bom can match during jlcpcb fab
Parts:
- C13: LCSC (none) -> C14663
- R3: LCSC (none) -> C22765
- U2: LCSC (none) -> C318884
Changed lines of the file:
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@@
+			)
+		)
+		(property "LCSC" "C318884"
+			(at 100.33 58.42 0)
+			(effects
+				(font
+					(size 1.27 1.27)
+				)
+				(hide yes)
 			)
 		)
@@
 			)
 		)
+		(property "LCSC" "C22765"
+			(at 133.35 53.34 0)
+			(effects
+				(font
+					(size 1.27 1.27)
+				)
+				(hide yes)
+			)
+		)
 		(pin "2"
 		)
@@
 			(at 21.59 27.94 0)
 			(effects
+				(font
+					(size 1.27 1.27)
+				)
+				(hide yes)
+			)
+		)
+		(property "LCSC" "C14663"
+			(at 21.59 27.94 0)
+			(effects
