File: usb.kicad_sch (KiCad schematic)
At the start: 5 parts, among them J43 USB_B, U24 USBLC6-2P6

Commit message: added lcsc field so that bom can match during jlcpcb fab
Parts:
- C76: LCSC (none) -> C14663
- D4: LCSC (none) -> C2297
- J43: LCSC (none) -> C456014
- R104: LCSC (none) -> C21190
- U24: LCSC (none) -> C15999
Changed lines of the file:
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@@
+			)
+		)
+		(property "LCSC" "C2297"
+			(at 96.52 62.23 90)
+			(effects
+				(font
+					(size 1.27 1.27)
+				)
+				(hide yes)
 			)
 		)
@@
 		)
 		(property "#" "C14663"
+			(at 121.92 54.61 0)
+			(effects
+				(font
+					(size 1.27 1.27)
+				)
+				(hide yes)
+			)
+		)
+		(property "LCSC" "C14663"
 			(at 121.92 54.61 0)
 			(effects
@@
 			)
 		)
+		(property "LCSC" "C456014"
+			(at 86.36 53.34 0)
+			(effects
+				(font
+					(size 1.27 1.27)
+				)
+				(hide yes)
+			)
+		)
 		(pin "1"
 		)
@@
 		)
 		(property "Tape" ""
+			(at 109.22 53.34 0)
+			(effects
+				(font
+					(size 1.27 1.27)
+				)
+				(hide yes)
+			)
+		)
+		(property "LCSC" "C15999"
 			(at 109.22 53.34 0)
 			(effects
@@
 			(at 96.52 69.85 0)
 			(effects
+				(font
+					(size 1.27 1.27)
+				)
+				(hide yes)
+			)
+		)
+		(property "LCSC" "C21190"
+			(at 96.52 69.85 0)
+			(effects
